Commit message: [FIX] Rename link name to make unique to avoid TF error

File: urdf/left_robot.xacro (robot description, xacro)
@@ -24,5 +24,5 @@
   </collision>
 </link>
-<link name="shoulder_1">
+<link name="left_shoulder">
   <inertial>
     <origin xyz="3.510374243868086e-17 0.02733088208948456 -2.220446049250313e-16" rpy="0 0 0"/>
@@ -44,5 +44,5 @@
   </collision>
 </link>
-<link name="upper_arm_1">
+<link name="left_upper_arm">
   <inertial>
     <origin xyz="0.008260426712845922 -5.551115123125783e-17 0.1430705592158692" rpy="0 0 0"/>
@@ -64,5 +64,5 @@
   </collision>
 </link>
-<link name="elbow_1">
+<link name="left_elbow">
   <inertial>
     <origin xyz="7.425709832186824e-17 9.070522111187529e-14 0.017967251502733594" rpy="0 0 0"/>
@@ -84,5 +84,5 @@
   </collision>
 </link>
-<link name="forearm_1">
+<link name="left_forearm">
   <inertial>
     <origin xyz="1.038890692768342e-16 -1.6653345369377348e-16 0.09502500346990606" rpy="0 0 0"/>
@@ -104,5 +104,5 @@
   </collision>
 </link>
-<link name="wrist_1">
+<link name="left_wrist">
   <inertial>
     <origin xyz="0.00022630011389308704 -5.662137425588298e-15 -0.014473720665364898" rpy="0 0 0"/>
@@ -124,5 +124,5 @@
   </collision>
 </link>
-<link name="hand_1">
+<link name="left_hand">
   <inertial>
     <origin xyz="0.015812535108693015 -2.7755575615628914e-16 4.241051954068098e-14" rpy="0 0 0"/>
@@ -144,5 +144,5 @@
   </collision>
 </link>
-<link name="upper_clamp_1">
+<link name="left_upper_clamp">
   <inertial>
     <origin xyz="0.03094811647250459 -0.0064395804078536956 0.0" rpy="0 0 0"/>
@@ -164,5 +164,5 @@
   </collision>
 </link>
-<link name="lower_clamp_1">
+<link name="left_lower_clamp">
   <inertial>
     <origin xyz="0.03039219722172494 0.0075333119271628335 0.0" rpy="0 0 0"/>
@@ -187,5 +187,5 @@
   <origin xyz="0.0 0.19651 1.3165" rpy="0 0 0"/>
   <parent link="base_link"/>
-  <child link="shoulder_1"/>
+  <child link="left_shoulder"/>
   <axis xyz="0.0 1.0 0.0"/>
   <limit upper="3.141593" lower="0.0" effort="100" velocity="100"/>
@@ -193,6 +193,6 @@
 <joint name="LJ2" type="revolute">
   <origin xyz="0.0 0.068 0.0" rpy="0 0 0"/>
-  <parent link="shoulder_1"/>
-  <child link="upper_arm_1"/>
+  <parent link="left_shoulder"/>
+  <child link="left_upper_arm"/>
   <axis xyz="-1.0 0.0 0.0"/>
   <limit upper="1.570796" lower="0.0" effort="100" velocity="100"/>
@@ -200,6 +200,6 @@
 <joint name="LJ3" type="revolute">
   <origin xyz="0.0 0.0 0.235" rpy="0 0 0"/>
-  <parent link="upper_arm_1"/>
-  <child link="elbow_1"/>
+  <parent link="left_upper_arm"/>
+  <child link="left_elbow"/>
   <axis xyz="0.0 0.0 1.0"/>
   <limit upper="3.141593" lower="0.0" effort="100" velocity="100"/>
@@ -207,6 +207,6 @@
 <joint name="LJ4" type="revolute">
   <origin xyz="0.0 0.0 0.039" rpy="0 0 0"/>
-  <parent link="elbow_1"/>
-  <child link="forearm_1"/>
+  <parent link="left_elbow"/>
+  <child link="left_forearm"/>
   <axis xyz="-1.0 -0.0 0.0"/>
   <limit upper="2.268928" lower="0.0" effort="100" velocity="100"/>
@@ -214,6 +214,6 @@
 <joint name="LJ5" type="revolute">
   <origin xyz="0.0 0.0 0.24" rpy="0 0 0"/>
-  <parent link="forearm_1"/>
-  <child link="wrist_1"/>
+  <parent link="left_forearm"/>
+  <child link="left_wrist"/>
   <axis xyz="0.0 -1.0 -0.0"/>
   <limit upper="3.141593" lower="0.0" effort="100" velocity="100"/>
@@ -221,6 +221,6 @@
 <joint name="LJ6" type="revolute">
   <origin xyz="0.023 0.0 0.0" rpy="0 0 0"/>
-  <parent link="wrist_1"/>
-  <child link="hand_1"/>
+  <parent link="left_wrist"/>
+  <child link="left_hand"/>
   <axis xyz="1.0 0.0 -0.0"/>
   <limit upper="3.141593" lower="0.0" effort="100" velocity="100"/>
@@ -228,6 +228,6 @@
 <joint name="LJ7" type="revolute">
   <origin xyz="0.025 -0.014 0.0" rpy="0 0 0"/>
-  <parent link="hand_1"/>
-  <child link="upper_clamp_1"/>
+  <parent link="left_hand"/>
+  <child link="left_upper_clamp"/>
   <axis xyz="-0.0 0.0 -1.0"/>
   <limit upper="1.22173" lower="0.0" effort="100" velocity="100"/>
@@ -235,6 +235,6 @@
 <joint name="LJ8" type="revolute">
   <origin xyz="0.025 0.014 0.0" rpy="0 0 0"/>
-  <parent link="hand_1"/>
-  <child link="lower_clamp_1"/>
+  <parent link="left_hand"/>
+  <child link="left_lower_clamp"/>
   <axis xyz="0.0 -0.0 1.0"/>
   <limit upper="1.22173" lower="0.0" effort="100" velocity="100"/>
